File: schematics/ESP_Display.kicad_sch (KiCad schematic)
At the start: 6 parts, among them U1 WeMos_S2_mini, U2 TXS0108EPW

Commit message: rename the project
Other:
- title: ESP HID Display -> ESP Display
Changed lines of the file:
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@@
 	(paper "A4")
 	(title_block
-		(title "ESP HID Display")
+		(title "ESP Display")
 	)
 	(junction
@@
 		)
 		(instances
-			(project "ESP_HID_Diplay"
+			(project "ESP_Display"
 				(path "/17b1ec26-ea5e-4607-9d09-c3e497ef61d1"
 					(reference "DS1")
@@
 		)
 		(instances
-			(project "ESP_HID_Diplay"
+			(project "ESP_Display"
 				(path "/17b1ec26-ea5e-4607-9d09-c3e497ef61d1"
 					(reference "U2")
@@
 		)
 		(instances
-			(project "ESP_HID_Diplay"
+			(project "ESP_Display"
 				(path "/17b1ec26-ea5e-4607-9d09-c3e497ef61d1"
 					(reference "RV1")
@@
 		)
 		(instances
-			(project "ESP_HID_Diplay"
+			(project "ESP_Display"
 				(path "/17b1ec26-ea5e-4607-9d09-c3e497ef61d1"
 					(reference "R1")
@@
 		)
 		(instances
-			(project "ESP_HID_Diplay"
+			(project "ESP_Display"
 				(path "/17b1ec26-ea5e-4607-9d09-c3e497ef61d1"
 					(reference "R2")
@@
 		)
 		(instances
-			(project "ESP_HID_Diplay"
+			(project "ESP_Display"
 				(path "/17b1ec26-ea5e-4607-9d09-c3e497ef61d1"
 					(reference "U1")
